File: Tarjeta-WiFi-control-techo.kicad_pcb (KiCad board)
At the start: 4 copper layers, 142 x 90 mm, 83 parts, among them J2 Conn_ARM_SWD_TagConnect_TC203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, J3 Conn_01x04_Pin, J4 Conn_01x02_Pin, J6 Conn_01x03_Socket, J7 Conn_01x09_Socket, Q2 BC817-40, Q3 BSS84P, SW1 SW_Push, U1 ESP32-WROOM-32E, U3 BH1750FVI-TR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

Commit message: Se agrego un conector para poder hacer uso del control manual
Parts:
- added J5: Conn_01x04_Socket, Connector_Phoenix_MC:PhoenixContact_MC_1,5_4-G-3.81_1x04_P3.81mm_Horizontal, F.Cu at (130.4, 134.9)
- moved R10 10.2 mm to (150.2, 136.3)
- moved TP2 10.2 mm to (151.2, 130.1)
- moved U3 10.2 mm to (155.3, 137.2)
- moved C5 10.2 mm to (154.1, 132.8)
- moved C6 10.2 mm to (157.1, 132.8)
- moved R11 10.2 mm to (147.5, 136.3)
Connections:
- net Net-(J7-Pin_6) renamed /BOT
- net Net-(J7-Pin_7) renamed /BTA
- net Net-(J7-Pin_8) renamed /BTF
Routing:
- net /BOT: track 16.9 -> 52.8 mm
- net /BTA: track 11.4 -> 36.7 mm
- net /BTF: track 11.8 -> 29.5 mm
- net /SDA: track 166.9 -> 177.8 mm
- net /DVI: track 161.4 -> 171.6 mm
- net /SCL: track 201.7 -> 211.5 mm
- added copper zone on B.Cu, net GNDREF

Commit message: final release
Parts:
- moved R9 119.7 mm to (201.7, 166.0), turned to 180 degrees
- moved C12 116.9 mm to (204.3, 91.2)
- moved C7 116.9 mm to (175.5, 167.8)
- moved C8 116.9 mm to (178.6, 167.8)
- moved J2 116.9 mm to (177.3, 148.1)
- moved J4 116.9 mm to (181.7, 124.9)
- moved R6 116.9 mm to (160.8, 118.6)
- moved TP1 116.9 mm to (266.3, 118.1)
- moved TP14 116.9 mm to (228.3, 145.7)
- moved TP15 116.9 mm to (237.9, 145.8)
- moved TP21 116.9 mm to (183.3, 165.7)
- moved TP7 116.9 mm to (166.8, 117.0)
- moved C15 116.9 mm to (155.8, 154.6)
- moved C3 116.9 mm to (155.8, 146.7)
- moved D2 116.9 mm to (163.5, 118.4)
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Routing:
- net /RS485-: track 20.6 -> 15.9 mm
- net /RS485+: track 20.6 -> 15.9 mm
- net /BOT: track 52.8 -> 48.8 mm
- net /SDA: track 177.8 -> 174.5 mm
- net Net-(J7-Pin_9): track 9.00 -> 11.8 mm
- net /DVI: track 171.6 -> 169.1 mm
- net /BTA: track 36.7 -> 34.6 mm
- net Net-(Q3-S): track 26.8 -> 25.4 mm
- net /BTF: track 29.5 -> 30.7 mm
- net /SCL: track 211.5 -> 210.3 mm
- net /AHT20_GND_CTRL: track 52.8 -> 54.0 mm
- net +12V: track 0.00 -> 0.90 mm
Other:
- outline, holes or cut-outs redrawn
- board text added: "NOTAS DE ENSAMBLE: 1. TODO EL PROCESO Y LA MANO DE OBRA DEBEN CUMPLIR CON LOS ESTÁNDARES IPC-A-610 Y J-STD-001, AMBOS CLASE 2. 2. SOLDADURA: [ELEGIR UNA OPCIÓN] A) PROCESO LIBRE DE PLOMO (ROHS) UTILIZANDO PASTA SAC305 O EQUIVALENTE. B) PROCESO CON PLOMO UTILIZANDO PASTA Sn63/Pb37. 3. LA COLOCACIÓN Y ORIENTACIÓN DE COMPONENTES DEBE BASARSE EN LA LISTA DE MATERIALES (BOM) REV. [Indicar Revisión] Y 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"
